File: WiiCamera/WiiCamera/WiiCameraSingleV2/WiicameraSingleV2.brd (EAGLE design)
At the start: 15.3 x 19 mm, 6 parts

Commit message: wii camera update
Routing:
- net GND: track 37.6 -> 43.9 mm, vias 3 -> 2
Changed lines of the file:
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@@
 <vertex x="0" y="0"/>
 </polygon>
-<wire x1="12.573" y1="16.129" x2="12.573" y2="12.954" width="0.6096" layer="16"/>
-<via x="12.573" y="12.954" extent="1-16" drill="0.6" shape="square"/>
-<wire x1="12.573" y1="12.954" x2="10.414" y2="12.954" width="0.6096" layer="1"/>
-<wire x1="10.414" y1="12.954" x2="10.287" y2="13.081" width="0.6096" layer="1"/>
 <wire x1="1.905" y1="16.129" x2="5.461" y2="16.129" width="0.6096" layer="16"/>
 <wire x1="5.461" y1="16.129" x2="5.969" y2="15.621" width="0.6096" layer="16"/>
@@
 <vertex x="0" y="0"/>
 </polygon>
+<wire x1="12.573" y1="16.129" x2="11.938" y2="16.129" width="0.4064" layer="16"/>
+<wire x1="11.938" y1="16.129" x2="10.541" y2="17.526" width="0.4064" layer="16"/>
+<wire x1="10.541" y1="17.526" x2="3.302" y2="17.526" width="0.4064" layer="16"/>
+<wire x1="3.302" y1="17.526" x2="1.905" y2="16.129" width="0.4064" layer="16"/>
 </signal>
 <signal name="SCL">
